File: Hardware/Z80BASE/Z80BASE.kicad_pcb (KiCad board)
At the start: 2 copper layers, 105 x 53 mm, 5 parts, among them J1 Conn_02x40_Odd_Even, J2 Conn_02x40_Odd_Even, J3 Conn_02x40_Odd_Even, J4 Conn_02x40_Odd_Even, J5 Conn_02x40_Odd_Even

Commit message: base ok
Connections:
- J1 pad 10: /HALT -> /RSV35
- J1 pad 12: /NMI -> /RSV34
- J1 pad 14: /INT -> /RSV33
- J1 pad 16: /RD -> /RSV32
- J1 pad 18: /WR -> /RSV31
- J1 pad 20: /BUSACK -> /RSV30
- J1 pad 22: /WAIT -> /RSV29
- J1 pad 24: /BUSRQ -> /RSV28
- J1 pad 26: /RESET -> /RSV27
- J1 pad 28: /M1 -> /RSV26
- J1 pad 30: /RFSH -> /RSV25
- J1 pad 32: /D0 -> /RSV24
- J1 pad 34: /D1 -> /RSV23
- J1 pad 36: /D2 -> /RSV22
- J1 pad 38: /D3 -> /RSV21
- J1 pad 40: /D4 -> /RSV20
- J1 pad 42: /D5 -> /RSV19
- J1 pad 44: /D6 -> /RSV18
- J1 pad 46: /D7 -> /RSV17
- J1 pad 48: /CLK -> /RSV16
- J1 pad 50: /A0 -> /RSV15
- J1 pad 52: /A1 -> /RSV14
- J1 pad 54: /A2 -> /RSV13
- J1 pad 56: /A3 -> /RSV12
- J1 pad 58: /A4 -> /RSV11
- J1 pad 6: /IORQ -> /RSV37
- J1 pad 60: /A5 -> /RSV10
- J1 pad 62: /A6 -> /RSV9
- J1 pad 64: /A7 -> /RSV8
- J1 pad 66: /A8 -> /RSV7
- J1 pad 68: /A9 -> /RSV6
- J1 pad 70: /A10 -> /RSV5
- J1 pad 72: /A11 -> /RSV4
- J1 pad 74: /A12 -> /RSV3
- J1 pad 76: /A13 -> /RSV2
- J1 pad 78: /A14 -> /RSV1
- J1 pad 8: /MREQ -> /RSV36
- J1 pad 80: /A15 -> /RSV0
- J2 pad 10: /A11 -> /RSV4
- J2 pad 12: /A10 -> /RSV5
- J2 pad 14: /A9 -> /RSV6
- J2 pad 16: /A8 -> /RSV7
- J2 pad 18: /A7 -> /RSV8
- J2 pad 2: /A15 -> /RSV0
- J2 pad 20: /A6 -> /RSV9
- J2 pad 22: /A5 -> /RSV10
- J2 pad 24: /A4 -> /RSV11
- J2 pad 26: /A3 -> /RSV12
- J2 pad 28: /A2 -> /RSV13
- J2 pad 30: /A1 -> /RSV14
- J2 pad 32: /A0 -> /RSV15
- J2 pad 34: /CLK -> /RSV16
- J2 pad 36: /D7 -> /RSV17
- J2 pad 38: /D6 -> /RSV18
- J2 pad 4: /A14 -> /RSV1
- J2 pad 40: /D5 -> /RSV19
- J2 pad 42: /D4 -> /RSV20
- J2 pad 44: /D3 -> /RSV21
- J2 pad 46: /D2 -> /RSV22
- J2 pad 48: /D1 -> /RSV23
- J2 pad 50: /D0 -> /RSV24
- J2 pad 52: /RFSH -> /RSV25
- J2 pad 54: /M1 -> /RSV26
- J2 pad 56: /RESET -> /RSV27
- J2 pad 58: /BUSRQ -> /RSV28
- J2 pad 6: /A13 -> /RSV2
- J2 pad 60: /WAIT -> /RSV29
- J2 pad 62: /BUSACK -> /RSV30
- J2 pad 64: /WR -> /RSV31
- J2 pad 66: /RD -> /RSV32
- J2 pad 68: /INT -> /RSV33
- J2 pad 70: /NMI -> /RSV34
- J2 pad 72: /HALT -> /RSV35
- J2 pad 74: /MREQ -> /RSV36
- J2 pad 76: /IORQ -> /RSV37
- J2 pad 8: /A12 -> /RSV3
- J3 pad 10: /A11 -> /RSV4
- J3 pad 12: /A10 -> /RSV5
- J3 pad 14: /A9 -> /RSV6
- J3 pad 16: /A8 -> /RSV7
- J3 pad 18: /A7 -> /RSV8
- J3 pad 2: /A15 -> /RSV0
- J3 pad 20: /A6 -> /RSV9
- J3 pad 22: /A5 -> /RSV10
- J3 pad 24: /A4 -> /RSV11
- J3 pad 26: /A3 -> /RSV12
- J3 pad 28: /A2 -> /RSV13
- J3 pad 30: /A1 -> /RSV14
- J3 pad 32: /A0 -> /RSV15
- J3 pad 34: /CLK -> /RSV16
- J3 pad 36: /D7 -> /RSV17
- J3 pad 38: /D6 -> /RSV18
- J3 pad 4: /A14 -> /RSV1
- J3 pad 40: /D5 -> /RSV19
- J3 pad 42: /D4 -> /RSV20
- J3 pad 44: /D3 -> /RSV21
- J3 pad 46: /D2 -> /RSV22
- J3 pad 48: /D1 -> /RSV23
- J3 pad 50: /D0 -> /RSV24
- J3 pad 52: /RFSH -> /RSV25
- J3 pad 54: /M1 -> /RSV26
- J3 pad 56: /RESET -> /RSV27
- J3 pad 58: /BUSRQ -> /RSV28
- J3 pad 6: /A13 -> /RSV2
- J3 pad 60: /WAIT -> /RSV29
- J3 pad 62: /BUSACK -> /RSV30
- J3 pad 64: /WR -> /RSV31
- J3 pad 66: /RD -> /RSV32
- J3 pad 68: /INT -> /RSV33
- J3 pad 70: /NMI -> /RSV34
- J3 pad 72: /HALT -> /RSV35
- J3 pad 74: /MREQ -> /RSV36
- J3 pad 76: /IORQ -> /RSV37
- J3 pad 8: /A12 -> /RSV3
- J4 pad 10: /A11 -> /RSV4
- J4 pad 12: /A10 -> /RSV5
- J4 pad 14: /A9 -> /RSV6
- J4 pad 16: /A8 -> /RSV7
- J4 pad 18: /A7 -> /RSV8
- J4 pad 2: /A15 -> /RSV0
- J4 pad 20: /A6 -> /RSV9
- J4 pad 22: /A5 -> /RSV10
- J4 pad 24: /A4 -> /RSV11
- J4 pad 26: /A3 -> /RSV12
- J4 pad 28: /A2 -> /RSV13
- J4 pad 30: /A1 -> /RSV14
- J4 pad 32: /A0 -> /RSV15
- J4 pad 34: /CLK -> /RSV16
- J4 pad 36: /D7 -> /RSV17
- J4 pad 38: /D6 -> /RSV18
- J4 pad 4: /A14 -> /RSV1
- J4 pad 40: /D5 -> /RSV19
- J4 pad 42: /D4 -> /RSV20
- J4 pad 44: /D3 -> /RSV21
- J4 pad 46: /D2 -> /RSV22
- J4 pad 48: /D1 -> /RSV23
- J4 pad 50: /D0 -> /RSV24
- J4 pad 52: /RFSH -> /RSV25
- J4 pad 54: /M1 -> /RSV26
- J4 pad 56: /RESET -> /RSV27
- J4 pad 58: /BUSRQ -> /RSV28
- J4 pad 6: /A13 -> /RSV2
- J4 pad 60: /WAIT -> /RSV29
- J4 pad 62: /BUSACK -> /RSV30
- J4 pad 64: /WR -> /RSV31
- J4 pad 66: /RD -> /RSV32
- J4 pad 68: /INT -> /RSV33
- J4 pad 70: /NMI -> /RSV34
- J4 pad 72: /HALT -> /RSV35
- J4 pad 74: /MREQ -> /RSV36
- J4 pad 76: /IORQ -> /RSV37
- J4 pad 8: /A12 -> /RSV3
- J5 pad 11: /NMI -> /RSV34
- J5 pad 13: /INT -> /RSV33
- J5 pad 15: /RD -> /RSV32
- J5 pad 17: /WR -> /RSV31
- J5 pad 19: /BUSACK -> /RSV30
- J5 pad 21: /WAIT -> /RSV29
- J5 pad 23: /BUSRQ -> /RSV28
- J5 pad 25: /RESET -> /RSV27
- J5 pad 27: /M1 -> /RSV26
- J5 pad 29: /RFSH -> /RSV25
- J5 pad 31: /D0 -> /RSV24
- J5 pad 33: /D1 -> /RSV23
- J5 pad 35: /D2 -> /RSV22
- J5 pad 37: /D3 -> /RSV21
- J5 pad 39: /D4 -> /RSV20
- J5 pad 41: /D5 -> /RSV19
- J5 pad 43: /D6 -> /RSV18
- J5 pad 45: /D7 -> /RSV17
- J5 pad 47: /CLK -> /RSV16
- J5 pad 49: /A0 -> /RSV15
- J5 pad 5: /IORQ -> /RSV37
- J5 pad 51: /A1 -> /RSV14
- J5 pad 53: /A2 -> /RSV13
- J5 pad 55: /A3 -> /RSV12
- J5 pad 57: /A4 -> /RSV11
- J5 pad 59: /A5 -> /RSV10
- J5 pad 61: /A6 -> /RSV9
- J5 pad 63: /A7 -> /RSV8
- J5 pad 65: /A8 -> /RSV7
- J5 pad 67: /A9 -> /RSV6
- J5 pad 69: /A10 -> /RSV5
- J5 pad 7: /MREQ -> /RSV36
- J5 pad 71: /A11 -> /RSV4
- J5 pad 73: /A12 -> /RSV3
- J5 pad 75: /A13 -> /RSV2
- J5 pad 77: /A14 -> /RSV1
- J5 pad 79: /A15 -> /RSV0
- J5 pad 9: /HALT -> /RSV35
Routing:
- net /WAIT: track 144.4 -> 49.5 mm
- net /RSV6: track 0.00 -> 49.6 mm
- net /RSV20: track 0.00 -> 49.6 mm
- net /RSV35: track 0.00 -> 49.6 mm
- net /RSV34: track 0.00 -> 49.6 mm
- net /RSV9: track 0.00 -> 49.5 mm
- net /RSV28: track 0.00 -> 49.5 mm
- net /RSV27: track 0.00 -> 49.5 mm
- net /RSV3: track 0.00 -> 49.5 mm
- net /RSV24: track 0.00 -> 49.5 mm
- net /RSV21: track 0.00 -> 49.5 mm
- net /RSV2: track 0.00 -> 49.5 mm
- net /RSV14: track 0.00 -> 49.5 mm
- net /RSV13: track 0.00 -> 49.5 mm
- net /RSV11: track 0.00 -> 49.5 mm
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Other:
- board text removed: "2019, ferreirasil.com"

Commit message: pcb project
Other:
- board text added: "www.ferreirasil.com"
